Commit message: Funcional

File: urdf/jetson_lidar_ed/parameters_jetson_lidar_ed_v1.xacro (robot description, xacro)
@@ -358,13 +358,13 @@
             <xacro:property name="lidar_pos_w" value="0.0"/>
     <!--Meshes -->
-        <xacro:property name="mesh_puzzlebot_chassis"  value="$(find puzzlebot_description)/meshes/bases/MCR2_puzzlebot_chassis_v1_2.stl" />
-        <xacro:property name="mesh_puzzlebot_motor_left"  value="$(find puzzlebot_description)/meshes/misc/MCR2_dc_motor_left.stl" />
-        <xacro:property name="mesh_puzzlebot_motor_right"  value="$(find puzzlebot_description)/meshes/misc/MCR2_dc_motor_right.stl" />
-        <xacro:property name="mesh_puzzlebot_wheel"  value="$(find puzzlebot_description)/meshes/wheels/MCR2_puzzlebot_wheel.stl" />
-        <xacro:property name="mesh_puzzlebot_caster"  value="$(find puzzlebot_description)/meshes/wheels/MCR2_puzzlebot_casterball.stl" />
-        <xacro:property name="mesh_puzzlebot_battery"  value="$(find puzzlebot_description)/meshes/misc/MCR2_puzzlebot_battery.stl" />
-        <xacro:property name="mesh_puzzlebot_jetson"  value="$(find puzzlebot_description)/meshes/misc/MCR2_nvidia_jetson_v1_2.stl" />
-        <xacro:property name="mesh_puzzlebot_camera"  value="$(find puzzlebot_description)/meshes/sensors/MCR2_puzzlebot_camera.stl" />
-        <xacro:property name="mesh_puzzlebot_lidar_base"  value="$(find puzzlebot_description)/meshes/bases/MCR2_puzzlebot_lidar_base_v1.stl" />
-        <xacro:property name="mesh_puzzlebot_lidar_sensor"  value="$(find puzzlebot_description)/meshes/sensors/MCR2_puzzlebot_lidar_sensor_v1.stl" />
+        <xacro:property name="mesh_puzzlebot_chassis"  value="$(find quetzalcoders_autonomousnavigation_puzzlebot)/meshes/bases/MCR2_puzzlebot_chassis_v1_2.stl" />
+        <xacro:property name="mesh_puzzlebot_motor_left"  value="$(find quetzalcoders_autonomousnavigation_puzzlebot)/meshes/misc/MCR2_dc_motor_left.stl" />
+        <xacro:property name="mesh_puzzlebot_motor_right"  value="$(find quetzalcoders_autonomousnavigation_puzzlebot)/meshes/misc/MCR2_dc_motor_right.stl" />
+        <xacro:property name="mesh_puzzlebot_wheel"  value="$(find quetzalcoders_autonomousnavigation_puzzlebot)/meshes/wheels/MCR2_puzzlebot_wheel.stl" />
+        <xacro:property name="mesh_puzzlebot_caster"  value="$(find quetzalcoders_autonomousnavigation_puzzlebot)/meshes/wheels/MCR2_puzzlebot_casterball.stl" />
+        <xacro:property name="mesh_puzzlebot_battery"  value="$(find quetzalcoders_autonomousnavigation_puzzlebot)/meshes/misc/MCR2_puzzlebot_battery.stl" />
+        <xacro:property name="mesh_puzzlebot_jetson"  value="$(find quetzalcoders_autonomousnavigation_puzzlebot)/meshes/misc/MCR2_nvidia_jetson_v1_2.stl" />
+        <xacro:property name="mesh_puzzlebot_camera"  value="$(find quetzalcoders_autonomousnavigation_puzzlebot)/meshes/sensors/MCR2_puzzlebot_camera.stl" />
+        <xacro:property name="mesh_puzzlebot_lidar_base"  value="$(find quetzalcoders_autonomousnavigation_puzzlebot)/meshes/bases/MCR2_puzzlebot_lidar_base_v1.stl" />
+        <xacro:property name="mesh_puzzlebot_lidar_sensor"  value="$(find quetzalcoders_autonomousnavigation_puzzlebot)/meshes/sensors/MCR2_puzzlebot_lidar_sensor_v1.stl" />
 </robot>

File: urdf/puzzlebot_jetson_lidar_ed_v1.xacro (robot description, xacro)
@@ -2,8 +2,8 @@
 <robot xmlns:xacro="http://www.ros.org/wiki/xacro" name="Puzzlebot_Hacker_Ed.">
 <!-- files for gazebo costumization -->
-<xacro:include filename="$(find puzzlebot_description)/urdf/jetson_lidar_ed/materials_jetson_lidar_ed.xacro" />
-<xacro:include filename="$(find puzzlebot_description)/urdf/jetson_lidar_ed/parameters_jetson_lidar_ed_v1.xacro" />
-<xacro:include filename="$(find puzzlebot_description)/urdf/jetson_lidar_ed/macros_jetson_lidar_ed.xacro" />
-<xacro:include filename="$(find puzzlebot_description)/urdf/jetson_lidar_ed/puzzlebot_jetson_lidar_ed_v1.gazebo.xacro" />
+<xacro:include filename="$(find quetzalcoders_autonomousnavigation_puzzlebot)/urdf/jetson_lidar_ed/materials_jetson_lidar_ed.xacro" />
+<xacro:include filename="$(find quetzalcoders_autonomousnavigation_puzzlebot)/urdf/jetson_lidar_ed/parameters_jetson_lidar_ed_v1.xacro" />
+<xacro:include filename="$(find quetzalcoders_autonomousnavigation_puzzlebot)/urdf/jetson_lidar_ed/macros_jetson_lidar_ed.xacro" />
+<xacro:include filename="$(find quetzalcoders_autonomousnavigation_puzzlebot)/urdf/jetson_lidar_ed/puzzlebot_jetson_lidar_ed_v1.gazebo.xacro" />
 <!--LINKS-->
 <!-- Dummy link to fix robot chassis -->
